File: KiCad/IoT/IoT.kicad_sch (KiCad schematic)
At the start: 57 parts, among them J1 USB_C_Receptacle_USB2.0_16P, J2 Program header, J3 Conn_01x08_Pin, J4 Micro_SD_Card_Det2, J5 Conn_01x08_Pin, J6 Flow sensor, SW1 SW_Push, SW2 SW_Push, SW3 SW_Push, SW4 SW_Push, SW5 SW_Push, U1 STM32F401RETx, Y1 32.768khz, Y2 HSE

Commit message: circuit bugfixes
Parts:
- added C13: 4.7u, symbol Device:C_Polarized
- added D17, D18: 3V3, symbol Device:D_Zener
- added D19, D20: PTVS5V0Z1USK, Diode_SMD:Nexperia_DSN1608-2_1.6x0.8mm, symbol Diode:PTVS5V0Z1USK
- added J2, J4, J7: Conn_01x01_Pin, symbol Connector:Conn_01x01_Pin
- added J3: Conn_01x04_Pin, symbol Connector:Conn_01x04_Pin
- added J5, J6: Conn_01x02_Pin, symbol Connector:Conn_01x02_Pin
- added J8: Conn_01x05_Pin, symbol Connector:Conn_01x05_Pin
- added J9: Conn_01x03_Pin, symbol Connector:Conn_01x03_Pin
- C2: renamed from C4; value 3p -> 18p
- C3: renamed from C5; value 3p -> 18p
- C4: renamed from C2; value 3p -> 7p
- C5: renamed from C3; value 3p -> 7p
- R7: value 18k -> 10k
- R8: value 10k -> 12k
- renumbered J2 to J10, J3 to J11, J4 to J12, J5 to J13, J6 to J14, Y2 to Y1, Y1 to Y2
Connections:
- net +3V3: now also U1.13 (VREF+), C13.1
- net GND: now also C13.2, D17.2 (A), D18.2 (A), D19.2 (A), D20.2 (A); no longer J1.A8 (SBU1), J1.B8 (SBU2)
- net I2C3_SCL: now also D17.1 (K)
- net I2C3_SDA: now also D18.1 (K)
- net LED1: now also U1.36 (PB15); no longer U1.39 (PC8)
- net USB_DM: now also D19.1 (K)
- net USB_DP: now also D20.1 (K)
- net at U1.10 (PC2): now also J3.3 (Pin_3)
- net at U1.11 (PC3): now also J3.4 (Pin_4)
- net at U1.14 (PA0): now also J5.1 (Pin_1)
- net at U1.15 (PA1): now also J5.2 (Pin_2)
- net at U1.2 (PC13): now also J4.1 (Pin_1)
- net at U1.26 (PB0): now also J8.1 (Pin_1)
- net at U1.27 (PB1): now also J8.2 (Pin_2)
- net at U1.28 (PB2): now also J8.3 (Pin_3)
- net at U1.29 (PB10): now also J9.3 (Pin_3)
- net at U1.42 (PA9): now also J6.1 (Pin_1)
- net at U1.43 (PA10): now also J6.2 (Pin_2)
- net at U1.50 (PA15): now also J7.1 (Pin_1)
- net at U1.54 (PD2): now also J2.1 (Pin_1)
- net at U1.55 (PB3): now also J8.4 (Pin_4)
- net at U1.56 (PB4): now also J8.5 (Pin_5)
- net at U1.61 (PB8): now also J9.1 (Pin_1)
- net at U1.62 (PB9): now also J9.2 (Pin_2)
- net at U1.8 (PC0): now also J3.1 (Pin_1)
- net at U1.9 (PC1): now also J3.2 (Pin_2)
Other:
- note added: "For digital pin"
- moved on the sheet: C2, C3, C4, C5, J11, J13, J14, R14, R15, Y1, Y2
