File: KiCad/IoT/RS232.kicad_sch (KiCad schematic)
At the start: 18 parts, among them IC1 MAX3222EAP+, IC2 MAX3222EAP+, J7 RS232_1, J8 RS232_1

Commit message: circuit bugfixes
Parts:
- renumbered C13 to C14, C14 to C15, C15 to C16, C16 to C17, C17 to C18, C18 to C19, C19 to C20, C20 to C21, C21 to C22, C22 to C23, J7 to J15, J8 to J16
Connections:
- net UART6_RX: now also IC1.13 (T1IN), IC2.13 (T1IN); no longer IC1.15 (R1OUT), IC2.15 (R1OUT)
- net UART6_TX: now also IC1.15 (R1OUT), IC2.15 (R1OUT); no longer IC1.13 (T1IN), IC2.13 (T1IN)
Other:
- moved on the sheet: J16, JP7, JP8
Changed lines of the file:
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@@
 	(wire
 		(pts
-			(xy 146.05 66.04) (xy 218.44 66.04)
+			(xy 146.05 66.04) (xy 219.71 66.04)
 		)
 		(stroke
@@
 	(wire
 		(pts
-			(xy 209.55 50.8) (xy 210.82 50.8)
+			(xy 210.82 50.8) (xy 212.09 50.8)
 		)
 		(stroke
@@
 	(wire
 		(pts
+			(xy 187.96 50.8) (xy 186.69 50.8)
+		)
+		(stroke
+			(width 0)
+			(type default)
+		)
+	)
+	(wire
+		(pts
 			(xy 45.72 46.99) (xy 45.72 49.53)
 		)
@@
 	(wire
 		(pts
-			(xy 209.55 45.72) (xy 210.82 45.72)
+			(xy 210.82 45.72) (xy 212.09 45.72)
 		)
 		(stroke
@@
 	(wire
 		(pts
-			(xy 198.12 50.8) (xy 199.39 50.8)
+			(xy 199.39 50.8) (xy 200.66 50.8)
 		)
 		(stroke
@@
 	(wire
 		(pts
-			(xy 198.12 48.26) (xy 198.12 50.8)
+			(xy 199.39 48.26) (xy 199.39 50.8)
 		)
 		(stroke
@@
 	(wire
 		(pts
-			(xy 210.82 60.96) (xy 200.66 60.96)
+			(xy 212.09 60.96) (xy 200.66 60.96)
 		)
 		(stroke
@@
 	(wire
 		(pts
-			(xy 186.69 45.72) (xy 199.39 45.72)
+			(xy 186.69 45.72) (xy 200.66 45.72)
 		)
 		(stroke
@@
 	(wire
 		(pts
-			(xy 186.69 48.26) (xy 198.12 48.26)
+			(xy 186.69 48.26) (xy 199.39 48.26)
 		)
 		(stroke
@@
 		)
 	)
+	(wire
+		(pts
+			(xy 187.96 55.88) (xy 186.69 55.88)
+		)
+		(stroke
+			(width 0)
+			(type default)
+		)
+	)
 	(hierarchical_label "UART6_TX"
 		(shape input)
-		(at 186.69 55.88 0)
+		(at 90.17 49.53 0)
 		(effects
 			(font
@@
 	(hierarchical_label "UART6_RX"
 		(shape input)
-		(at 90.17 49.53 0)
+		(at 187.96 55.88 0)
 		(effects
 			(font
@@
 	(hierarchical_label "UART6_TX"
 		(shape input)
-		(at 90.17 54.61 0)
+		(at 187.96 50.8 0)
 		(effects
 			(font
@@
 	(hierarchical_label "UART6_RX"
 		(shape input)
-		(at 186.69 50.8 0)
+		(at 90.17 54.61 0)
 		(effects
 			(font
@@
 		(in_pos_files yes)
 		(dnp no)
-		(property "Reference" "C21"
+		(property "Reference" "C22"
 			(at 147.32 39.624 90)
 			(show_name no)
@@
 			(project "IoT"
 				(path "/f5d15b22-d91e-4545-b7af-da23c1769042/43c31ab3-a50b-4c6f-a99c-c41c2f249985"
-					(reference "C21")
+					(reference "C22")
 					(unit 1)
 				)
@@
 		(in_pos_files yes)
 		(dnp no)
-		(property "Reference" "C22"
+		(property "Reference" "C23"
 			(at 147.066 46.99 90)
 			(show_name no)
@@
 			(project "IoT"
 				(path "/f5d15b22-d91e-4545-b7af-da23c1769042/43c31ab3-a50b-4c6f-a99c-c41c2f249985"
-					(reference "C22")
+					(reference "C23")
 					(unit 1)
 				)
@@
 		(in_pos_files yes)
 		(dnp no)
-		(property "Reference" "C13"
+		(property "Reference" "C14"
 			(at 40.132 36.322 0)
 			(show_name no)
@@
 			(project "IoT"
 				(path "/f5d15b22-d91e-4545-b7af-da23c1769042/43c31ab3-a50b-4c6f-a99c-c41c2f249985"
-					(reference "C13")
+					(reference "C14")
 					(unit 1)
 				)
@@
 		(in_pos_files yes)
 		(dnp no)
-		(property "Reference" "C15"
+		(property "Reference" "C16"
 			(at 47.752 59.182 0)
 			(show_name no)
@@
 			(project "IoT"
 				(path "/f5d15b22-d91e-4545-b7af-da23c1769042/43c31ab3-a50b-4c6f-a99c-c41c2f249985"
-					(reference "C15")
+					(reference "C16")
 					(unit 1)
 				)
@@
 		(in_pos_files yes)
 		(dnp no)
-		(property "Reference" "C19"
+		(property "Reference" "C20"
 			(at 137.922 50.292 0)
 			(show_name no)
@@
 			(project "IoT"
 				(path "/f5d15b22-d91e-4545-b7af-da23c1769042/43c31ab3-a50b-4c6f-a99c-c41c2f249985"
-					(reference "C19")
+					(reference "C20")
 					(unit 1)
 				)
@@
 		(in_pos_files yes)
 		(dnp no)
-		(property "Reference" "C14"
+		(property "Reference" "C15"
 			(at 40.132 49.022 0)
 			(show_name no)
@@
 			(project "IoT"
 				(path "/f5d15b22-d91e-4545-b7af-da23c1769042/43c31ab3-a50b-4c6f-a99c-c41c2f249985"
-					(reference "C14")
+					(reference "C15")
 					(unit 1)
 				)
@@
 		(in_pos_files yes)
 		(dnp no)
-		(property "Reference" "C20"
+		(property "Reference" "C21"
 			(at 145.542 60.452 0)
 			(show_name no)
@@
 			(project "IoT"
 				(path "/f5d15b22-d91e-4545-b7af-da23c1769042/43c31ab3-a50b-4c6f-a99c-c41c2f249985"
-					(reference "C20")
+					(reference "C21")
 					(unit 1)
 				)
@@
 	(symbol
 		(lib_id "Connector:DE9_Socket_MountingHoles")
-		(at 218.44 50.8 0)
+		(at 219.71 50.8 0)
 		(unit 1)
 		(body_style 1)
@@
 		(in_pos_files yes)
 		(dnp no)
-		(property "Reference" "J8"
-			(at 217.424 35.306 0)
+		(property "Reference" "J16"
+			(at 218.694 35.306 0)
 			(show_name no)
 			(do_not_autoplace no)
@@
 		)
 		(property "Value" "RS232_1"
-			(at 218.948 63.246 0)
+			(at 220.218 63.246 0)
 			(show_name no)
 			(do_not_autoplace no)
@@
 		)
 		(property "Footprint" "Connector_Dsub:DSUB-9_Pins_Horizontal_P2.77x2.84mm_EdgePinOffset14.56mm_Housed_MountingHolesOffset15.98mm"
-			(at 218.44 50.8 0)
+			(at 219.71 50.8 0)
 			(hide yes)
 			(show_name no)
@@
 		)
 		(property "Datasheet" ""
-			(at 218.44 50.8 0)
+			(at 219.71 50.8 0)
 			(hide yes)
 			(show_name no)
@@
 		)
 		(property "Description" "9-pin D-SUB connector, socket (female), Mounting Hole"
-			(at 218.44 50.8 0)
+			(at 219.71 50.8 0)
 			(hide yes)
 			(show_name no)
@@
 			(project "IoT"
 				(path "/f5d15b22-d91e-4545-b7af-da23c1769042/43c31ab3-a50b-4c6f-a99c-c41c2f249985"
-					(reference "J8")
+					(reference "J16")
 					(unit 1)
 				)
@@
 		(in_pos_files yes)
 		(dnp no)
-		(property "Reference" "C18"
+		(property "Reference" "C19"
 			(at 137.922 37.592 0)
 			(show_name no)
@@
 			(project "IoT"
 				(path "/f5d15b22-d91e-4545-b7af-da23c1769042/43c31ab3-a50b-4c6f-a99c-c41c2f249985"
-					(reference "C18")
+					(reference "C19")
 					(unit 1)
 				)
@@
 		(in_pos_files yes)
 		(dnp no)
-		(property "Reference" "J7"
+		(property "Reference" "J15"
 			(at 119.634 34.036 0)
 			(show_name no)
@@
 			(project "IoT"
 				(path "/f5d15b22-d91e-4545-b7af-da23c1769042/43c31ab3-a50b-4c6f-a99c-c41c2f249985"
-					(reference "J7")
+					(reference "J15")
 					(unit 1)
 				)
@@
 	(symbol
 		(lib_id "Jumper:SolderJumper_2_Open")
-		(at 204.47 50.8 0)
+		(at 205.74 50.8 0)
 		(unit 1)
 		(body_style 1)
@@
 		(dnp no)
 		(property "Reference" "JP8"
-			(at 204.47 48.768 0)
+			(at 205.74 48.768 0)
 			(show_name no)
 			(do_not_autoplace no)
@@
 		)
 		(property "Value" "SolderJumper_2_Open"
-			(at 204.47 46.99 0)
+			(at 205.74 46.99 0)
 			(hide yes)
 			(show_name no)
@@
 		)
 		(property "Footprint" "Package_SON:WSON-8-1EP_6x5mm_P1.27mm_EP3.4x4mm"
-			(at 204.47 50.8 0)
+			(at 205.74 50.8 0)
 			(hide yes)
 			(show_name no)
@@
 		)
 		(property "Datasheet" ""
-			(at 204.47 58.42 0)
+			(at 205.74 58.42 0)
 			(hide yes)
 			(show_name no)
@@
 		)
 		(property "Description" "Solder Jumper, 2-pole, open"
-			(at 204.47 55.88 0)
+			(at 205.74 55.88 0)
 			(hide yes)
 			(show_name no)
@@
 	(symbol
 		(lib_id "Jumper:SolderJumper_2_Open")
-		(at 204.47 45.72 0)
+		(at 205.74 45.72 0)
 		(unit 1)
 		(body_style 1)
@@
 		(dnp no)
 		(property "Reference" "JP7"
-			(at 204.47 43.942 0)
+			(at 205.74 43.942 0)
 			(show_name no)
 			(do_not_autoplace no)
@@
 		)
 		(property "Value" "SolderJumper_2_Open"
-			(at 204.47 41.91 0)
+			(at 205.74 41.91 0)
 			(hide yes)
 			(show_name no)
@@
 		)
 		(property "Footprint" "Package_SON:WSON-8-1EP_6x5mm_P1.27mm_EP3.4x4mm"
-			(at 204.47 45.72 0)
+			(at 205.74 45.72 0)
 			(hide yes)
 			(show_name no)
@@
 		)
 		(property "Datasheet" ""
-			(at 204.47 53.34 0)
+			(at 205.74 53.34 0)
 			(hide yes)
 			(show_name no)
@@
 		)
 		(property "Description" "Solder Jumper, 2-pole, open"
-			(at 204.47 50.8 0)
+			(at 205.74 50.8 0)
 			(hide yes)
 			(show_name no)
@@
 		(in_pos_files yes)
 		(dnp no)
-		(property "Reference" "C16"
+		(property "Reference" "C17"
 			(at 49.53 38.354 90)
 			(show_name no)
@@
 			(project "IoT"
 				(path "/f5d15b22-d91e-4545-b7af-da23c1769042/43c31ab3-a50b-4c6f-a99c-c41c2f249985"
-					(reference "C16")
+					(reference "C17")
 					(unit 1)
 				)
@@
 		(in_pos_files yes)
 		(dnp no)
-		(property "Reference" "C17"
+		(property "Reference" "C18"
 			(at 49.276 45.72 90)
 			(show_name no)
@@
 			(project "IoT"
 				(path "/f5d15b22-d91e-4545-b7af-da23c1769042/43c31ab3-a50b-4c6f-a99c-c41c2f249985"
-					(reference "C17")
+					(reference "C18")
 					(unit 1)
 				)
